File: Buffers_Out.kicad_sch (KiCad schematic)
At the start: 29 parts, among them U4 MCP6002-xSN, X1 PEDAL_COMBO_TOP

Commit message: Input buffer and power
Updated the input buffer layout.
Updated the power supply layout.
Parts:
- C22: renamed from C24; footprint Capacitor_SMD:C_1206_3216Metric -> Capacitor_SMD:C_0805_2012Metric
- C23: renamed from C25; footprint Capacitor_SMD:C_1206_3216Metric -> Capacitor_SMD:C_0805_2012Metric
- renumbered C20 to C18, C21 to C19, C22 to C20, C23 to C21, C26 to C24, C27 to C25, C28 to C26
Connections:
- net FILT_RP: now reaches R14.2, R16.1, R20.1
- net OPP_L: now reaches C18.1, R18.2, U4.3 (+)
- net OPO_L: now reaches C20.2, C22.1, R21.2, U4.1
- net OPM_L: now reaches C20.1, R17.2, U4.2 (-)
- net FILT_LM: now reaches R11.2, R17.1, R21.1
- net OPP_R: now reaches C19.1, R20.2, U4.5 (+)
- net FILT_LP: now reaches R12.2, R15.1, R18.1
- net FILT_RM: now reaches R13.2, R19.1, R22.1
- net OPO_R: now reaches C21.2, C23.1, R22.2, U4.7
- net OPM_R: now reaches C21.1, R19.2, U4.6 (-)
Other:
- moved on the sheet: C18, C19, C20, C21, C22, C23, C24, C25, D5, D6, R11, R12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
