File: Hardware/Power.kicad_sch (KiCad schematic)
At the start: 23 parts, among them U1 AMS1117-5.0, U2 AMS1117-3.3, X1 PEDAL_COMBO_TOP

Commit message: Build materials
Uploaded all files required for assembly.
Parts:
- FB1, FB2, FB3: value 300 -> 850
Changed lines of the file:
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@@
 			)
 		)
-		(property "Value" "300"
+		(property "Value" "850"
 			(at 184.15 46.99 90)
 			(show_name no)
@@
 			)
 		)
-		(property "Value" "300"
+		(property "Value" "850"
 			(at 194.31 113.03 90)
 			(show_name no)
@@
 			)
 		)
-		(property "Value" "300"
+		(property "Value" "850"
 			(at 129.54 44.45 90)
 			(show_name no)
