File: Hardware/Power.kicad_sch (KiCad schematic)
At the start: 23 parts, among them U1 AMS1117-5.0, U2 AMS1117-3.3, X1 PEDAL_COMBO_TOP

Commit message: Layout revision
Minor updated to references.
Minor updated to the PCB layout.
Parts:
- renumbered C8 to C10, C7 to C11, C9 to C12, C42 to C13, C10 to C14, C41 to C2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
