File: Hardware/Buffers_Out.kicad_sch (KiCad schematic)
At the start: 29 parts, among them U4 MCP6002-xSN, X1 PEDAL_COMBO_TOP

Commit message: Layout revision
Minor updated to references.
Minor updated to the PCB layout.
Parts:
- renumbered C18 to C22, C19 to C23, C20 to C24, C21 to C25, C22 to C26, C23 to C27, C24 to C28, C25 to C29, C26 to C30
Changed lines of the file:
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@@
 		(dnp no)
 		(fields_autoplaced yes)
-		(property "Reference" "C18"
+		(property "Reference" "C22"
 			(at 97.79 69.8499 0)
 			(show_name no)
@@
 			(project "PicoFX"
 				(path "/4cbf131b-42e8-4a05-beea-68c6d66cdb1a/f30b69e3-f4a5-44b3-bff9-cd489323ac3e"
-					(reference "C18")
+					(reference "C22")
 					(unit 1)
 				)
@@
 		(in_pos_files yes)
 		(dnp no)
-		(property "Reference" "#PWR039"
+		(property "Reference" "#PWR042"
 			(at 137.16 146.05 0)
 			(hide yes)
@@
 			(project "PicoFX"
 				(path "/4cbf131b-42e8-4a05-beea-68c6d66cdb1a/f30b69e3-f4a5-44b3-bff9-cd489323ac3e"
-					(reference "#PWR039")
+					(reference "#PWR042")
 					(unit 1)
 				)
@@
 		(in_pos_files yes)
 		(dnp no)
-		(property "Reference" "#PWR040"
+		(property "Reference" "#PWR043"
 			(at 147.32 76.2 0)
 			(hide yes)
@@
 			(project "PicoFX"
 				(path "/4cbf131b-42e8-4a05-beea-68c6d66cdb1a/f30b69e3-f4a5-44b3-bff9-cd489323ac3e"
-					(reference "#PWR040")
+					(reference "#PWR043")
 					(unit 1)
 				)
@@
 		(in_pos_files yes)
 		(dnp no)
-		(property "Reference" "#PWR038"
+		(property "Reference" "#PWR041"
 			(at 137.16 76.2 0)
 			(hide yes)
@@
 			(project "PicoFX"
 				(path "/4cbf131b-42e8-4a05-beea-68c6d66cdb1a/f30b69e3-f4a5-44b3-bff9-cd489323ac3e"
-					(reference "#PWR038")
+					(reference "#PWR041")
 					(unit 1)
 				)
@@
 		(dnp no)
 		(fields_autoplaced yes)
-		(property "Reference" "#PWR044"
+		(property "Reference" "#PWR047"
 			(at 203.2 81.28 0)
 			(hide yes)
@@
 			(project "PicoFX"
 				(path "/4cbf131b-42e8-4a05-beea-68c6d66cdb1a/f30b69e3-f4a5-44b3-bff9-cd489323ac3e"
-					(reference "#PWR044")
+					(reference "#PWR047")
 					(unit 1)
 				)
@@
 		(in_pos_files yes)
 		(dnp no)
-		(property "Reference" "#PWR042"
+		(property "Reference" "#PWR045"
 			(at 157.48 76.2 0)
 			(hide yes)
@@
 			(project "PicoFX"
 				(path "/4cbf131b-42e8-4a05-beea-68c6d66cdb1a/f30b69e3-f4a5-44b3-bff9-cd489323ac3e"
-					(reference "#PWR042")
+					(reference "#PWR045")
 					(unit 1)
 				)
@@
 		(in_pos_files yes)
 		(dnp no)
-		(property "Reference" "#PWR043"
+		(property "Reference" "#PWR046"
 			(at 157.48 146.05 0)
 			(hide yes)
@@
 			(project "PicoFX"
 				(path "/4cbf131b-42e8-4a05-beea-68c6d66cdb1a/f30b69e3-f4a5-44b3-bff9-cd489323ac3e"
-					(reference "#PWR043")
+					(reference "#PWR046")
 					(unit 1)
 				)
@@
 		(dnp no)
 		(fields_autoplaced yes)
-		(property "Reference" "C19"
+		(property "Reference" "C23"
 			(at 97.79 139.6999 0)
 			(show_name no)
@@
 			(project "PicoFX"
 				(path "/4cbf131b-42e8-4a05-beea-68c6d66cdb1a/f30b69e3-f4a5-44b3-bff9-cd489323ac3e"
-					(reference "C19")
+					(reference "C23")
 					(unit 1)
 				)
@@
 		(in_pos_files yes)
 		(dnp no)
-		(property "Reference" "C26"
+		(property "Reference" "C30"
 			(at 191.77 88.8999 0)
 			(show_name no)
@@
 			(project "PicoFX"
 				(path "/4cbf131b-42e8-4a05-beea-68c6d66cdb1a/f30b69e3-f4a5-44b3-bff9-cd489323ac3e"
-					(reference "C26")
+					(reference "C30")
 					(unit 1)
 				)
@@
 		(dnp no)
 		(fields_autoplaced yes)
-		(property "Reference" "C24"
+		(property "Reference" "C28"
 			(at 151.13 62.2299 0)
 			(show_name no)
@@
 			(project "PicoFX"
 				(path "/4cbf131b-42e8-4a05-beea-68c6d66cdb1a/f30b69e3-f4a5-44b3-bff9-cd489323ac3e"
-					(reference "C24")
+					(reference "C28")
 					(unit 1)
 				)
@@
 		(in_pos_files yes)
 		(dnp no)
-		(property "Reference" "C20"
+		(property "Reference" "C24"
 			(at 104.14 40.64 90)
 			(show_name no)
@@
 			(project "PicoFX"
 				(path "/4cbf131b-42e8-4a05-beea-68c6d66cdb1a/f30b69e3-f4a5-44b3-bff9-cd489323ac3e"
-					(reference "C20")
+					(reference "C24")
 					(unit 1)
 				)
@@
 		(dnp no)
 		(fields_autoplaced yes)
-		(property "Reference" "C25"
+		(property "Reference" "C29"
 			(at 151.13 132.0799 0)
 			(show_name no)
@@
 			(project "PicoFX"
 				(path "/4cbf131b-42e8-4a05-beea-68c6d66cdb1a/f30b69e3-f4a5-44b3-bff9-cd489323ac3e"
-					(reference "C25")
+					(reference "C29")
 					(unit 1)
 				)
@@
 		(in_pos_files yes)
 		(dnp no)
-		(property "Reference" "C21"
+		(property "Reference" "C25"
 			(at 104.14 110.49 90)
 			(show_name no)
@@
 			(project "PicoFX"
 				(path "/4cbf131b-42e8-4a05-beea-68c6d66cdb1a/f30b69e3-f4a5-44b3-bff9-cd489323ac3e"
-					(reference "C21")
+					(reference "C25")
 					(unit 1)
 				)
@@
 		(dnp no)
 		(fields_autoplaced yes)
-		(property "Reference" "C23"
+		(property "Reference" "C27"
 			(at 120.65 119.38 90)
 			(show_name no)
@@
 			(project "PicoFX"
 				(path "/4cbf131b-42e8-4a05-beea-68c6d66cdb1a/f30b69e3-f4a5-44b3-bff9-cd489323ac3e"
-					(reference "C23")
+					(reference "C27")
 					(unit 1)
 				)
@@
 		(in_pos_files yes)
 		(dnp no)
-		(property "Reference" "#PWR041"
+		(property "Reference" "#PWR044"
 			(at 147.32 146.05 0)
 			(hide yes)
@@
 			(project "PicoFX"
 				(path "/4cbf131b-42e8-4a05-beea-68c6d66cdb1a/f30b69e3-f4a5-44b3-bff9-cd489323ac3e"
-					(reference "#PWR041")
+					(reference "#PWR044")
 					(unit 1)
 				)
@@
 		(dnp no)
 		(fields_autoplaced yes)
-		(property "Reference" "C22"
+		(property "Reference" "C26"
 			(at 120.65 49.53 90)
 			(show_name no)
@@
 			(project "PicoFX"
 				(path "/4cbf131b-42e8-4a05-beea-68c6d66cdb1a/f30b69e3-f4a5-44b3-bff9-cd489323ac3e"
-					(reference "C22")
+					(reference "C26")
 					(unit 1)
 				)
@@
 		(dnp no)
 		(fields_autoplaced yes)
-		(property "Reference" "#PWR045"
+		(property "Reference" "#PWR048"
 			(at 203.2 109.22 0)
 			(hide yes)
@@
 			(project "PicoFX"
 				(path "/4cbf131b-42e8-4a05-beea-68c6d66cdb1a/f30b69e3-f4a5-44b3-bff9-cd489323ac3e"
-					(reference "#PWR045")
+					(reference "#PWR048")
 					(unit 1)
 				)
@@
 		(dnp no)
 		(fields_autoplaced yes)
-		(property "Reference" "#PWR046"
+		(property "Reference" "#PWR049"
 			(at 247.65 104.14 0)
 			(hide yes)
@@
 			(project "PicoFX"
 				(path "/4cbf131b-42e8-4a05-beea-68c6d66cdb1a/f30b69e3-f4a5-44b3-bff9-cd489323ac3e"
-					(reference "#PWR046")
-					(unit 1)
-				)
+					(reference "#PWR049")
+					(unit 1)
+				)
