File: Hardware/Codec.kicad_sch (KiCad schematic)
At the start: 17 parts, among them U5 CS4272

Commit message: Layout revision
Minor updated to references.
Minor updated to the PCB layout.
Parts:
- renumbered C27 to C31, C28 to C32, C29 to C33, C30 to C34, C31 to C35, C32 to C36, C33 to C37, C34 to C38, C35 to C39, C36 to C40, C37 to C41, C38 to C42
Changed lines of the file:
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@@
 		(dnp no)
 		(fields_autoplaced yes)
-		(property "Reference" "#PWR050"
+		(property "Reference" "#PWR053"
 			(at 102.87 53.34 0)
 			(hide yes)
@@
 			(project "PicoFX"
 				(path "/4cbf131b-42e8-4a05-beea-68c6d66cdb1a/f7920eb9-f1f4-4882-8d74-32484732cce5"
-					(reference "#PWR050")
+					(reference "#PWR053")
 					(unit 1)
 				)
@@
 		(in_pos_files yes)
 		(dnp no)
-		(property "Reference" "C33"
+		(property "Reference" "C37"
 			(at 163.83 73.6599 0)
 			(show_name no)
@@
 			(project "PicoFX"
 				(path "/4cbf131b-42e8-4a05-beea-68c6d66cdb1a/f7920eb9-f1f4-4882-8d74-32484732cce5"
-					(reference "C33")
+					(reference "C37")
 					(unit 1)
 				)
@@
 		(dnp no)
 		(fields_autoplaced yes)
-		(property "Reference" "#PWR052"
+		(property "Reference" "#PWR055"
 			(at 102.87 104.14 0)
 			(hide yes)
@@
 			(project "PicoFX"
 				(path "/4cbf131b-42e8-4a05-beea-68c6d66cdb1a/f7920eb9-f1f4-4882-8d74-32484732cce5"
-					(reference "#PWR052")
+					(reference "#PWR055")
 					(unit 1)
 				)
@@
 		(dnp no)
 		(fields_autoplaced yes)
-		(property "Reference" "#PWR060"
+		(property "Reference" "#PWR063"
 			(at 187.96 88.9 0)
 			(hide yes)
@@
 			(project "PicoFX"
 				(path "/4cbf131b-42e8-4a05-beea-68c6d66cdb1a/f7920eb9-f1f4-4882-8d74-32484732cce5"
-					(reference "#PWR060")
+					(reference "#PWR063")
 					(unit 1)
 				)
@@
 		(in_pos_files yes)
 		(dnp no)
-		(property "Reference" "C34"
+		(property "Reference" "C38"
 			(at 163.83 83.8201 0)
 			(show_name no)
@@
 			(project "PicoFX"
 				(path "/4cbf131b-42e8-4a05-beea-68c6d66cdb1a/f7920eb9-f1f4-4882-8d74-32484732cce5"
-					(reference "C34")
+					(reference "C38")
 					(unit 1)
 				)
@@
 		(in_pos_files yes)
 		(dnp no)
-		(property "Reference" "C28"
+		(property "Reference" "C32"
 			(at 106.68 73.6599 0)
 			(show_name no)
@@
 			(project "PicoFX"
 				(path "/4cbf131b-42e8-4a05-beea-68c6d66cdb1a/f7920eb9-f1f4-4882-8d74-32484732cce5"
-					(reference "C28")
+					(reference "C32")
 					(unit 1)
 				)
@@
 		(dnp no)
 		(fields_autoplaced yes)
-		(property "Reference" "#PWR051"
+		(property "Reference" "#PWR054"
 			(at 102.87 72.39 0)
 			(hide yes)
@@
 			(project "PicoFX"
 				(path "/4cbf131b-42e8-4a05-beea-68c6d66cdb1a/f7920eb9-f1f4-4882-8d74-32484732cce5"
-					(reference "#PWR051")
+					(reference "#PWR054")
 					(unit 1)
 				)
@@
 		(dnp no)
 		(fields_autoplaced yes)
-		(property "Reference" "#PWR048"
+		(property "Reference" "#PWR051"
 			(at 93.98 88.9 0)
 			(hide yes)
@@
 			(project "PicoFX"
 				(path "/4cbf131b-42e8-4a05-beea-68c6d66cdb1a/f7920eb9-f1f4-4882-8d74-32484732cce5"
-					(reference "#PWR048")
+					(reference "#PWR051")
 					(unit 1)
 				)
@@
 		(in_pos_files yes)
 		(dnp no)
-		(property "Reference" "C27"
+		(property "Reference" "C31"
 			(at 106.68 54.6099 0)
 			(show_name no)
@@
 			(project "PicoFX"
 				(path "/4cbf131b-42e8-4a05-beea-68c6d66cdb1a/f7920eb9-f1f4-4882-8d74-32484732cce5"
-					(reference "C27")
+					(reference "C31")
 					(unit 1)
 				)
@@
 		(dnp no)
 		(fields_autoplaced yes)
-		(property "Reference" "#PWR061"
+		(property "Reference" "#PWR064"
 			(at 187.96 116.84 0)
 			(hide yes)
@@
 			(project "PicoFX"
 				(path "/4cbf131b-42e8-4a05-beea-68c6d66cdb1a/f7920eb9-f1f4-4882-8d74-32484732cce5"
-					(reference "#PWR061")
+					(reference "#PWR064")
 					(unit 1)
 				)
@@
 		(dnp no)
 		(fields_autoplaced yes)
-		(property "Reference" "#PWR056"
+		(property "Reference" "#PWR059"
 			(at 177.8 116.84 0)
 			(hide yes)
@@
 			(project "PicoFX"
 				(path "/4cbf131b-42e8-4a05-beea-68c6d66cdb1a/f7920eb9-f1f4-4882-8d74-32484732cce5"
-					(reference "#PWR056")
+					(reference "#PWR059")
 					(unit 1)
 				)
@@
 		(dnp no)
 		(fields_autoplaced yes)
-		(property "Reference" "#PWR055"
+		(property "Reference" "#PWR058"
 			(at 165.1 144.78 0)
 			(hide yes)
@@
 			(project "PicoFX"
 				(path "/4cbf131b-42e8-4a05-beea-68c6d66cdb1a/f7920eb9-f1f4-4882-8d74-32484732cce5"
-					(reference "#PWR055")
+					(reference "#PWR058")
 					(unit 1)
 				)
@@
 		(in_pos_files yes)
 		(dnp no)
-		(property "Reference" "C29"
+		(property "Reference" "C33"
 			(at 119.38 54.6099 0)
 			(show_name no)
@@
 			(project "PicoFX"
 				(path "/4cbf131b-42e8-4a05-beea-68c6d66cdb1a/f7920eb9-f1f4-4882-8d74-32484732cce5"
-					(reference "C29")
+					(reference "C33")
 					(unit 1)
 				)
@@
 		(dnp no)
 		(fields_autoplaced yes)
-		(property "Reference" "#PWR057"
+		(property "Reference" "#PWR060"
 			(at 177.8 144.78 0)
 			(hide yes)
@@
 			(project "PicoFX"
 				(path "/4cbf131b-42e8-4a05-beea-68c6d66cdb1a/f7920eb9-f1f4-4882-8d74-32484732cce5"
-					(reference "#PWR057")
+					(reference "#PWR060")
 					(unit 1)
 				)
@@
 		(dnp no)
 		(fields_autoplaced yes)
-		(property "Reference" "#PWR054"
+		(property "Reference" "#PWR057"
 			(at 139.7 144.78 0)
 			(hide yes)
@@
 			(project "PicoFX"
 				(path "/4cbf131b-42e8-4a05-beea-68c6d66cdb1a/f7920eb9-f1f4-4882-8d74-32484732cce5"
-					(reference "#PWR054")
+					(reference "#PWR057")
 					(unit 1)
 				)
@@
 		(dnp no)
 		(fields_autoplaced yes)
-		(property "Reference" "#PWR058"
+		(property "Reference" "#PWR061"
 			(at 179.07 53.34 0)
 			(hide yes)
@@
 			(project "PicoFX"
 				(path "/4cbf131b-42e8-4a05-beea-68c6d66cdb1a/f7920eb9-f1f4-4882-8d74-32484732cce5"
-					(reference "#PWR058")
+					(reference "#PWR061")
 					(unit 1)
 				)
@@
 		(dnp no)
 		(fields_autoplaced yes)
-		(property "Reference" "#PWR053"
+		(property "Reference" "#PWR056"
 			(at 119.38 144.78 0)
 			(hide yes)
@@
 			(project "PicoFX"
 				(path "/4cbf131b-42e8-4a05-beea-68c6d66cdb1a/f7920eb9-f1f4-4882-8d74-32484732cce5"
-					(reference "#PWR053")
+					(reference "#PWR056")
 					(unit 1)
 				)
@@
 		(dnp no)
 		(fields_autoplaced yes)
-		(property "Reference" "#PWR059"
+		(property "Reference" "#PWR062"
 			(at 187.96 69.85 0)
 			(hide yes)
@@
 			(project "PicoFX"
 				(path "/4cbf131b-42e8-4a05-beea-68c6d66cdb1a/f7920eb9-f1f4-4882-8d74-32484732cce5"
-					(reference "#PWR059")
+					(reference "#PWR062")
 					(unit 1)
 				)
@@
 		(in_pos_files yes)
 		(dnp no)
-		(property "Reference" "C32"
+		(property "Reference" "C36"
 			(at 170.18 54.6101 0)
 			(show_name no)
@@
 			(project "PicoFX"
 				(path "/4cbf131b-42e8-4a05-beea-68c6d66cdb1a/f7920eb9-f1f4-4882-8d74-32484732cce5"
-					(reference "C32")
+					(reference "C36")
 					(unit 1)
 				)
@@
 		(dnp no)
 		(fields_autoplaced yes)
-		(property "Reference" "#PWR047"
+		(property "Reference" "#PWR050"
 			(at 93.98 69.85 0)
 			(hide yes)
@@
 			(project "PicoFX"
 				(path "/4cbf131b-42e8-4a05-beea-68c6d66cdb1a/f7920eb9-f1f4-4882-8d74-32484732cce5"
-					(reference "#PWR047")
+					(reference "#PWR050")
 					(unit 1)
 				)
@@
 		(in_pos_files yes)
 		(dnp no)
-		(property "Reference" "C30"
+		(property "Reference" "C34"
 			(at 119.38 73.6599 0)
 			(show_name no)
@@
 			(project "PicoFX"
 				(path "/4cbf131b-42e8-4a05-beea-68c6d66cdb1a/f7920eb9-f1f4-4882-8d74-32484732cce5"
-					(reference "C30")
+					(reference "C34")
 					(unit 1)
 				)
@@
 		(in_pos_files yes)
 		(dnp no)
-		(property "Reference" "C35"
+		(property "Reference" "C39"
 			(at 173.99 128.2699 0)
 			(show_name no)
@@
 			(project "PicoFX"
 				(path "/4cbf131b-42e8-4a05-beea-68c6d66cdb1a/f7920eb9-f1f4-4882-8d74-32484732cce5"
-					(reference "C35")
+					(reference "C39")
 					(unit 1)
 				)
@@
 		(in_pos_files yes)
 		(dnp no)
-		(property "Reference" "C38"
+		(property "Reference" "C42"
 			(at 176.53 83.8201 0)
 			(show_name no)
@@
 			(project "PicoFX"
 				(path "/4cbf131b-42e8-4a05-beea-68c6d66cdb1a/f7920eb9-f1f4-4882-8d74-32484732cce5"
-					(reference "C38")
+					(reference "C42")
 					(unit 1)
 				)
@@
 		(dnp no)
 		(fields_autoplaced yes)
-		(property "Reference" "#PWR049"
+		(property "Reference" "#PWR052"
 			(at 93.98 104.14 0)
 			(hide yes)
@@
 			(project "PicoFX"
 				(path "/4cbf131b-42e8-4a05-beea-68c6d66cdb1a/f7920eb9-f1f4-4882-8d74-32484732cce5"
-					(reference "#PWR049")
+					(reference "#PWR052")
 					(unit 1)
 				)
@@
 		(in_pos_files yes)
 		(dnp no)
-		(property "Reference" "C36"
+		(property "Reference" "C40"
 			(at 182.88 54.6101 0)
 			(show_name no)
@@
 			(project "PicoFX"
 				(path "/4cbf131b-42e8-4a05-beea-68c6d66cdb1a/f7920eb9-f1f4-4882-8d74-32484732cce5"
-					(reference "C36")
+					(reference "C40")
 					(unit 1)
 				)
@@
 		(in_pos_files yes)
 		(dnp no)
-		(property "Reference" "C31"
+		(property "Reference" "C35"
 			(at 161.29 128.2699 0)
 			(show_name no)
@@
 			(project "PicoFX"
 				(path "/4cbf131b-42e8-4a05-beea-68c6d66cdb1a/f7920eb9-f1f4-4882-8d74-32484732cce5"
-					(reference "C31")
+					(reference "C35")
 					(unit 1)
 				)
@@
 		(in_pos_files yes)
 		(dnp no)
-		(property "Reference" "C37"
+		(property "Reference" "C41"
 			(at 176.53 73.6599 0)
 			(show_name no)
@@
 			(project "PicoFX"
 				(path "/4cbf131b-42e8-4a05-beea-68c6d66cdb1a/f7920eb9-f1f4-4882-8d74-32484732cce5"
-					(reference "C37")
-					(unit 1)
-				)
+					(reference "C41")
+					(unit 1)
+				)
